Commit message: Clean Go2 extreme-parkour: teacher PPO + DAgger student, remove GHN/NAS

File: legged_gym/resources/robots/go2/urdf/go2_with_camera.urdf (robot description, URDF)
Before this commit: robot go2_description, 30 links, 29 joints
Joints:
- joint d435i_camera_joint: origin xyz=0.34 -0.00 0.08 rpy=0 0.45 0 -> xyz=0.34 -0.00 0.09 rpy=0 0.0 0

Commit message: clean go2 working

File: legged_gym/resources/robots/go2/urdf/go2_with_camera.urdf (robot description, URDF)
Before this commit: robot go2_description, 30 links, 29 joints
Links:
- link d435i_camera: geometry 
Joints:
- joint d435i_camera_joint: origin xyz=0.34 -0.00 0.09 rpy=0 0.0 0 -> xyz=0.34 -0.00 0.09 rpy=0 0.00 0
